Commit message: update simulation parameters

File: f450_description/scripts/f450_robot/robot.urdf (robot description, URDF)
Before this commit: robot f450_uav, 9 links, 8 joints
Links:
- removed link base_link
- removed link battery_link
- removed link body_link
- removed link imu_link
- removed link raspberry_pi_link
- removed link rotor_1_link
- removed link rotor_2_link
- removed link rotor_3_link
- removed link rotor_4_link
- added link bottom_plate, mass 1.25653; collision mesh filename=package://f450_description/assets/1045_propeller.stl; collision mesh filename=package://f450_description/assets/1045_propeller.stl
Joints:
- removed joint base_to_body
- removed joint body_to_battery
- removed joint body_to_imu
- removed joint body_to_raspberry_pi
- removed joint body_to_rotor_1
- removed joint body_to_rotor_2
- removed joint body_to_rotor_3
- removed joint body_to_rotor_4

File: f450_description/urdf/f450_base.xacro (robot description, xacro)
@@ -13,12 +13,13 @@
     <inertial>
       <origin xyz="0 0 0" rpy="0 0 0"/>
-      <mass value="1.09429"/>
+      <mass value="1.25653"/>
       <inertia
-        ixx="0.0108413"
-        ixy="2.4413e-06"
-        ixz="3.72834e-05"
-        iyy="0.011469"
-        iyz="-3.48279e-06"
-        izz="0.0199678"/>
+      ixx="0.012363"
+      ixy="3.3165e-05"
+      ixz="5.60471e-05"
+      iyy="0.0124502"
+      iyz="-0.00031169"
+      izz="0.0213427"
+      />
     </inertial>
   </link>
@@ -27,5 +28,5 @@
     <parent link="base_link"/>
     <child link="body_link"/>
-    <origin xyz="0 0 0" rpy="0 0 0"/>
+    <origin xyz="-0.0653685 0.0328291 0" rpy="0 0 0"/>
   </joint>
 </robot>

File: f450_description/urdf/f450_frames.xacro (robot description, xacro)
@@ -25,35 +25,151 @@
             rpy="0 0 -3.14159"/>
   </joint>
-  <!-- Rotor 1 -->
-  <link name="rotor_1_link"/>
-  <joint name="body_to_rotor_1" type="fixed">
+  <!-- Camera frame -->
+  <link name="camera_link"/>
+  <joint name="body_to_camera" type="fixed">
+    <parent link="body_link"/>
+    <child link="camera_link"/>
+    <origin xyz="0.0528721 -0.106185 -0.0215468"
+            rpy="-1.5708 0 0"/>
+  </joint>
+  <!--
+    Rotor 1 joint.
+    Front-left rotor.
+    Rotation direction: CCW.
+    Continuous joint is required by the Gazebo multicopter
+    motor model plugin.
+    Rotor axis:
+      +Z body axis
+  -->
+  <link name="rotor_1_link">
+    <inertial>
+      <origin xyz="0 0 0" rpy="0 0 0"/>
+      <mass value="0.015"/>
+      <inertia
+        ixx="1.0e-05"
+        ixy="0.0"
+        ixz="0.0"
+        iyy="1.0e-05"
+        iyz="0.0"
+        izz="2.0e-05"/>
+    </inertial>
+  </link>
+  <joint name="body_to_rotor_1" type="continuous">
     <parent link="body_link"/>
     <child link="rotor_1_link"/>
     <origin xyz="-0.0935326 0.126083 0.0744345"
             rpy="0 0 1.5708"/>
+    <axis xyz="0 0 1"/>
+    <limit
+      effort="100.0"
+      velocity="2000.0"/>
+    <dynamics
+      damping="0.0"
+      friction="0.0"/>
   </joint>
-  <!-- Rotor 2 -->
-  <link name="rotor_2_link"/>
-  <joint name="body_to_rotor_2" type="fixed">
+  <!--
+    Rotor 2 joint.
+    Front-right rotor.
+    Rotation direction: CW.
+    Continuous joint is required by the Gazebo multicopter
+    motor model plugin.
+    Rotor axis:
+      +Z body axis
+  -->
+  <link name="rotor_2_link">
+    <inertial>
+      <origin xyz="0 0 0" rpy="0 0 0"/>
+      <mass value="0.015"/>
+      <inertia
+        ixx="1.0e-05"
+        ixy="0.0"
+        ixz="0.0"
+        iyy="1.0e-05"
+        iyz="0.0"
+        izz="2.0e-05"/>
+    </inertial>
+  </link>
+  <joint name="body_to_rotor_2" type="continuous">
     <parent link="body_link"/>
     <child link="rotor_2_link"/>
     <origin xyz="0.22428 0.126072 0.0744345"
             rpy="0 0 0"/>
+    <axis xyz="0 0 1"/>
+    <limit
+      effort="100.0"
+      velocity="2000.0"/>
+    <dynamics
+      damping="0.0"
+      friction="0.0"/>
   </joint>
-  <!-- Rotor 3 -->
-  <link name="rotor_3_link"/>
-  <joint name="body_to_rotor_3" type="fixed">
+  <!--
+    Rotor 3 joint.
+    Rear-right rotor.
+    Rotation direction: CCW.
+    Continuous joint is required by the Gazebo multicopter
+    motor model plugin.
+    Rotor axis:
+      +Z body axis
+  -->
+  <link name="rotor_3_link">
+    <inertial>
+      <origin xyz="0 0 0" rpy="0 0 0"/>
+      <mass value="0.015"/>
+      <inertia
+        ixx="1.0e-05"
+        ixy="0.0"
+        ixz="0.0"
+        iyy="1.0e-05"
+        iyz="0.0"
+        izz="2.0e-05"/>
+    </inertial>
+  </link>
+  <joint name="body_to_rotor_3" type="continuous">
     <parent link="body_link"/>
     <child link="rotor_3_link"/>
     <origin xyz="0.22427 -0.191741 0.0744345"
             rpy="0 0 -1.5708"/>
+    <axis xyz="0 0 1"/>
+    <limit
+      effort="100.0"
+      velocity="2000.0"/>
+    <dynamics
+      damping="0.0"
+      friction="0.0"/>
   </joint>
-  <!-- Rotor 4 -->
-  <link name="rotor_4_link"/>
-  <joint name="body_to_rotor_4" type="fixed">
+  <!--
+    Rotor 4 joint.
+    Rear-left rotor.
+    Rotation direction: CW.
+    Continuous joint is required by the Gazebo multicopter
+    motor model plugin.
+    Rotor axis:
+      +Z body axis
+  -->
+  <link name="rotor_4_link">
+    <inertial>
+      <origin xyz="0 0 0" rpy="0 0 0"/>
+      <mass value="0.015"/>
+      <inertia
+        ixx="1.0e-05"
+        ixy="0.0"
+        ixz="0.0"
+        iyy="1.0e-05"
+        iyz="0.0"
+        izz="2.0e-05"/>
+    </inertial>
+  </link>
+  <joint name="body_to_rotor_4" type="continuous">
     <parent link="body_link"/>
     <child link="rotor_4_link"/>
     <origin xyz="-0.0935433 -0.19173 0.0744345"
             rpy="0 0 -3.14159"/>
+    <axis xyz="0 0 1"/>
+    <limit
+      effort="100.0"
+      velocity="2000.0"/>
+    <dynamics
+      damping="0.0"
+      friction="0.0"/>
   </joint>
 </robot>

File: f450_description/urdf/f450_gazebo.xacro (robot description, xacro)
@@ -61,5 +61,26 @@
     </sensor>
   </gazebo>
-  <!-- Rotor frame markers for future multirotor plugin -->
+  <!-- Camera sensor attached to camera_link -->
+  <gazebo reference="camera_link">
+    <sensor name="camera_sensor" type="camera">
+      <always_on>true</always_on>
+      <update_rate>30</update_rate>
+      <visualize>true</visualize>
+      <topic>/f450/camera/image</topic>
+      <camera>
+        <horizontal_fov>1.047</horizontal_fov>
+        <image>
+          <width>640</width>
+          <height>480</height>
+          <format>R8G8B8</format>
+        </image>
+        <clip>
+          <near>0.05</near>
+          <far>100.0</far>
+        </clip>
+      </camera>
+    </sensor>
+  </gazebo>
+  <!-- Rotor visual/material tags -->
   <gazebo reference="rotor_1_link">
     <material>Gazebo/Blue</material>
@@ -74,3 +95,195 @@
     <material>Gazebo/Blue</material>
   </gazebo>
+  <!--
+    ============================================================================
+    F450 Multirotor Motor Model Configuration
+    ============================================================================
+    Rotor layout (top view):
+              Front (+X)
+          rotor_1       rotor_2
+             CCW           CW
+          rotor_4       rotor_3
+              CW          CCW
+              Rear (-X)
+    Motor and propeller setup:
+      - Motor: 2212 920KV
+      - Propeller: 9.4x4.3
+      - Battery: 3S LiPo (11.1V)
+    Experimental measurements with propeller:
+      RPM_max ≈ 7900 rpm
+    Angular velocity conversion:
+      omega = RPM * 2*pi / 60
+      omega_max =
+        7900 * 2*pi / 60
+      omega_max ≈ 827 rad/s
+    Estimated maximum thrust:
+      T_max ≈ 700 gf
+      T_max ≈ 6.8647 N
+    Rotor thrust model:
+      T = k_f * omega^2
+    Therefore:
+      k_f = T_max / omega_max^2
+      k_f =
+        6.8647 / 827^2
+      k_f ≈ 1.00e-05 N.s^2/rad^2
+    Hover estimation:
+      vehicle mass = 1.25653 kg
+      vehicle weight:
+        W = m * g
+        W = 12.32 N
+      hover thrust per rotor:
+        T_hover = W / 4
+        T_hover ≈ 3.08 N
+      hover angular velocity:
+        omega_hover =
+          sqrt(T_hover / k_f)
+        omega_hover ≈ 555 rad/s
+    Notes:
+      - These values are first-order estimates.
+      - Parameters should later be calibrated with a real thrust stand.
+      - Increased time constants improve simulation realism and stability.
+    ============================================================================
+  -->
+  <!-- Shared motor parameters -->
+  <xacro:property name="motor_time_constant_up" value="0.08"/>
+  <xacro:property name="motor_time_constant_down" value="0.12"/>
+  <xacro:property name="motor_max_rot_velocity" value="827.0"/>
+  <xacro:property name="motor_constant" value="1.00e-05"/>
+  <xacro:property name="motor_moment_constant" value="0.012"/>
+  <xacro:property name="rotor_drag_coefficient" value="8.0e-05"/>
+  <xacro:property name="rolling_moment_coefficient" value="1.0e-06"/>
+  <xacro:property name="rotor_velocity_slowdown_sim" value="10"/>
+  <!-- Rotor 1: front-left, CCW -->
+  <gazebo>
+    <plugin
+      filename="libignition-gazebo6-multicopter-motor-model-system.so"
+      name="ignition::gazebo::systems::MulticopterMotorModel">
+      <robotNamespace>f450_uav</robotNamespace>
+      <jointName>body_to_rotor_1</jointName>
+      <linkName>rotor_1_link</linkName>
+      <motorNumber>0</motorNumber>
+      <turningDirection>ccw</turningDirection>
+      <timeConstantUp>${motor_time_constant_up}</timeConstantUp>
+      <timeConstantDown>${motor_time_constant_down}</timeConstantDown>
+      <maxRotVelocity>${motor_max_rot_velocity}</maxRotVelocity>
+      <motorConstant>${motor_constant}</motorConstant>
+      <momentConstant>${motor_moment_constant}</momentConstant>
+      <commandSubTopic>command/motor_speed</commandSubTopic>
+      <motorSpeedPubTopic>motor_speed/0</motorSpeedPubTopic>
+      <rotorDragCoefficient>
+        ${rotor_drag_coefficient}
+      </rotorDragCoefficient>
+      <rollingMomentCoefficient>
+        ${rolling_moment_coefficient}
+      </rollingMomentCoefficient>
+      <rotorVelocitySlowdownSim>
+        ${rotor_velocity_slowdown_sim}
+      </rotorVelocitySlowdownSim>
+      <motorType>velocity</motorType>
+    </plugin>
+  </gazebo>
+  <!-- Rotor 2: front-right, CW -->
+  <gazebo>
+    <plugin
+      filename="libignition-gazebo6-multicopter-motor-model-system.so"
+      name="ignition::gazebo::systems::MulticopterMotorModel">
+      <robotNamespace>f450_uav</robotNamespace>
+      <jointName>body_to_rotor_2</jointName>
+      <linkName>rotor_2_link</linkName>
+      <motorNumber>1</motorNumber>
+      <turningDirection>cw</turningDirection>
+      <timeConstantUp>${motor_time_constant_up}</timeConstantUp>
+      <timeConstantDown>${motor_time_constant_down}</timeConstantDown>
+      <maxRotVelocity>${motor_max_rot_velocity}</maxRotVelocity>
+      <motorConstant>${motor_constant}</motorConstant>
+      <momentConstant>${motor_moment_constant}</momentConstant>
+      <commandSubTopic>command/motor_speed</commandSubTopic>
+      <motorSpeedPubTopic>motor_speed/1</motorSpeedPubTopic>
+      <rotorDragCoefficient>
+        ${rotor_drag_coefficient}
+      </rotorDragCoefficient>
+      <rollingMomentCoefficient>
+        ${rolling_moment_coefficient}
+      </rollingMomentCoefficient>
+      <rotorVelocitySlowdownSim>
+        ${rotor_velocity_slowdown_sim}
+      </rotorVelocitySlowdownSim>
+      <motorType>velocity</motorType>
+    </plugin>
+  </gazebo>
+  <!-- Rotor 3: rear-right, CCW -->
+  <gazebo>
+    <plugin
+      filename="libignition-gazebo6-multicopter-motor-model-system.so"
+      name="ignition::gazebo::systems::MulticopterMotorModel">
+      <robotNamespace>f450_uav</robotNamespace>
+      <jointName>body_to_rotor_3</jointName>
+      <linkName>rotor_3_link</linkName>
+      <motorNumber>2</motorNumber>
+      <turningDirection>ccw</turningDirection>
+      <timeConstantUp>${motor_time_constant_up}</timeConstantUp>
+      <timeConstantDown>${motor_time_constant_down}</timeConstantDown>
+      <maxRotVelocity>${motor_max_rot_velocity}</maxRotVelocity>
+      <motorConstant>${motor_constant}</motorConstant>
+      <momentConstant>${motor_moment_constant}</momentConstant>
+      <commandSubTopic>command/motor_speed</commandSubTopic>
+      <motorSpeedPubTopic>motor_speed/2</motorSpeedPubTopic>
+      <rotorDragCoefficient>
+        ${rotor_drag_coefficient}
+      </rotorDragCoefficient>
+      <rollingMomentCoefficient>
+        ${rolling_moment_coefficient}
+      </rollingMomentCoefficient>
+      <rotorVelocitySlowdownSim>
+        ${rotor_velocity_slowdown_sim}
+      </rotorVelocitySlowdownSim>
+      <motorType>velocity</motorType>
+    </plugin>
+  </gazebo>
+  <!-- Rotor 4: rear-left, CW -->
+  <gazebo>
+    <plugin
+      filename="libignition-gazebo6-multicopter-motor-model-system.so"
+      name="ignition::gazebo::systems::MulticopterMotorModel">
+      <robotNamespace>f450_uav</robotNamespace>
+      <jointName>body_to_rotor_4</jointName>
+      <linkName>rotor_4_link</linkName>
+      <motorNumber>3</motorNumber>
+      <turningDirection>cw</turningDirection>
+      <timeConstantUp>${motor_time_constant_up}</timeConstantUp>
+      <timeConstantDown>${motor_time_constant_down}</timeConstantDown>
+      <maxRotVelocity>${motor_max_rot_velocity}</maxRotVelocity>
+      <motorConstant>${motor_constant}</motorConstant>
+      <momentConstant>${motor_moment_constant}</momentConstant>
+      <commandSubTopic>command/motor_speed</commandSubTopic>
+      <motorSpeedPubTopic>motor_speed/3</motorSpeedPubTopic>
+      <rotorDragCoefficient>
+        ${rotor_drag_coefficient}
+      </rotorDragCoefficient>
+      <rollingMomentCoefficient>
+        ${rolling_moment_coefficient}
+      </rollingMomentCoefficient>
+      <rotorVelocitySlowdownSim>
+        ${rotor_velocity_slowdown_sim}
+      </rotorVelocitySlowdownSim>
+      <motorType>velocity</motorType>
+    </plugin>
+  </gazebo>
 </robot>
+<!-- My tests were as follows.
+No Load.
+M1 = .47A, 10,400rpm, 11.67 V, 891 Kv.
+M2 = .54A, 10,450 rpm, 11.73V, 890 Kv.
+M3 = .50A, 10,200rpm, 11.62V, 878 Kv.
+M4 = .44A, 10,150, rpm, 11.58V, 876Kv.
+With Stock propeller DJi 9.4 x 4.3
+Mi = 8.14A, 7,800rpm, 11.36 V,% NLS. 77.1
+M2 = 8.28A, 7,900 rpm, 11.40 V,% NLS. 77.9
+M3 = 7.86A, 7,900rpm, 11.31 V,% NLS. 79.6
+M4 = 7.79A, 7,800, rpm, 11.28 V,% NLS.78.9
+This motor is not you can put bigger prop because even with this motorine is quite hot, but not enough to consider not accelerate fully.
+Practically this limit in its 94 watts.
+94 watts between weight 50 grams is 1.88 watts per gram.
+Nothing to do with what many brands claim 3 or 4 watts per gram.
+In multicopters, 2 to 2.4 watts per gram is much longer.
+Avoid overheating to eliminate accidents.  -->

File: f450_description/urdf/f450_meshes.xacro (robot description, xacro)
@@ -50,4 +50,20 @@
       </geometry>
     </collision>
+    <!-- Part camera_support -->
+    <visual>
+      <origin xyz="0.0658056 -0.104579 -0.0032165" rpy="0 0 -3.14159"/>
+      <geometry>
+        <mesh filename="package://f450_description/meshes/camera_support.stl"/>
+      </geometry>
+      <material name="camera_support_material">
+        <color rgba="0.25098 0.25098 0.25098 1"/>
+      </material>
+    </visual>
+    <collision>
+      <origin xyz="0.0658056 -0.104579 -0.0032165" rpy="0 0 -3.14159"/>
+      <geometry>
+        <mesh filename="package://f450_description/meshes/camera_support.stl"/>
+      </geometry>
+    </collision>
     <!-- Part mpu_9250 -->
     <visual>
@@ -162,4 +178,20 @@
       </geometry>
     </collision>
+    <!-- Part leg -->
+    <visual>
+      <origin xyz="0.0183105 0.00715784 -0.000217496" rpy="-3.14159 0 0.785398"/>
+      <geometry>
+        <mesh filename="package://f450_description/meshes/leg.stl"/>
+      </geometry>
+      <material name="leg_material">
+        <color rgba="0.25098 0.25098 0.25098 1"/>
+      </material>
+    </visual>
+    <collision>
+      <origin xyz="0.0183105 0.00715784 -0.000217496" rpy="-3.14159 0 0.785398"/>
+      <geometry>
+        <mesh filename="package://f450_description/meshes/leg.stl"/>
+      </geometry>
+    </collision>
     <!-- Part top_plate -->
     <visual>
@@ -290,4 +322,20 @@
       </geometry>
     </collision>
+    <!-- Part logitech_c270b -->
+    <visual>
+      <origin xyz="0.0528721 -0.106185 -0.0215468" rpy="-1.5708 -0 0"/>
+      <geometry>
+        <mesh filename="package://f450_description/meshes/logitech_c270b.stl"/>
+      </geometry>
+      <material name="logitech_c270b_material">
+        <color rgba="0.294118 0.294118 0.294118 1"/>
+      </material>
+    </visual>
+    <collision>
+      <origin xyz="0.0528721 -0.106185 -0.0215468" rpy="-1.5708 -0 0"/>
+      <geometry>
+        <mesh filename="package://f450_description/meshes/logitech_c270b.stl"/>
+      </geometry>
+    </collision>
     <!-- Part holybro_brushless_motor_2216_880kv_3 -->
     <visual>
@@ -306,4 +354,20 @@
       </geometry>
     </collision>
+    <!-- Part leg_2 -->
+    <visual>
+      <origin xyz="0.105355 0.0142289 -0.000217496" rpy="-3.14159 -0 -0.785398"/>
+      <geometry>
+        <mesh filename="package://f450_description/meshes/leg.stl"/>
+      </geometry>
+      <material name="leg_2_material">
+        <color rgba="0.25098 0.25098 0.25098 1"/>
+      </material>
+    </visual>
+    <collision>
+      <origin xyz="0.105355 0.0142289 -0.000217496" rpy="-3.14159 -0 -0.785398"/>
+      <geometry>
+        <mesh filename="package://f450_description/meshes/leg.stl"/>
+      </geometry>
+    </collision>
     <!-- Part holybro_brushless_motor_2216_880kv_4 -->
     <visual>
@@ -322,4 +386,36 @@
       </geometry>
     </collision>
+    <!-- Part leg_3 -->
+    <visual>
+      <origin xyz="0.0253816 -0.079887 -0.000217496" rpy="-3.14159 0 2.35619"/>
+      <geometry>
+        <mesh filename="package://f450_description/meshes/leg.stl"/>
+      </geometry>
+      <material name="leg_3_material">
+        <color rgba="0.25098 0.25098 0.25098 1"/>
+      </material>
+    </visual>
+    <collision>
+      <origin xyz="0.0253816 -0.079887 -0.000217496" rpy="-3.14159 0 2.35619"/>
+      <geometry>
+        <mesh filename="package://f450_description/meshes/leg.stl"/>
+      </geometry>
+    </collision>
+    <!-- Part logitech_c270c -->
+    <visual>
+      <origin xyz="0.0528721 -0.0398885 -0.011086" rpy="1.74533 -0 0"/>
+      <geometry>
+        <mesh filename="package://f450_description/meshes/logitech_c270c.stl"/>
+      </geometry>
+      <material name="logitech_c270c_material">
+        <color rgba="0.294118 0.294118 0.294118 1"/>
+      </material>
+    </visual>
+    <collision>
+      <origin xyz="0.0528721 -0.0398885 -0.011086" rpy="1.74533 -0 0"/>
+      <geometry>
+        <mesh filename="package://f450_description/meshes/logitech_c270c.stl"/>
+      </geometry>
+    </collision>
     <!-- Part arm_4 -->
     <visual>
@@ -354,4 +450,20 @@
       </geometry>
     </collision>
+    <!-- Part leg_4 -->
+    <visual>
+      <origin xyz="0.112426 -0.0728159 -0.000217496" rpy="-3.14159 -0 -2.35619"/>
+      <geometry>
+        <mesh filename="package://f450_description/meshes/leg.stl"/>
+      </geometry>
+      <material name="leg_4_material">
+        <color rgba="0.25098 0.25098 0.25098 1"/>
+      </material>
+    </visual>
+    <collision>
+      <origin xyz="0.112426 -0.0728159 -0.000217496" rpy="-3.14159 -0 -2.35619"/>
+      <geometry>
+        <mesh filename="package://f450_description/meshes/leg.stl"/>
+      </geometry>
+    </collision>
     <!-- Part littlebee_spring30a_3 -->
     <visual>
